Commit message: "added ros2 controllers, launch files and gazeb"

File: reaction_wheel_pendulum_description/reaction_wheel_pendulum/robot.urdf.xacro (robot description, xacro)
@@ -1,3 +1,5 @@
-<robot name="reaction_wheel_pendulum">
+<?xml version="1.0"?>
+<robot name="reaction_wheel_pendulum" xmlns:xacro="http://wiki.ros.org/xacro">
+<xacro:include filename="$(find reaction_wheel_pendulum_description)/reaction_wheel_pendulum/ros2_control.urdf.xacro"/>
 <link name="support_plaform_1">
 <visual>
@@ -140,5 +142,5 @@
 </inertial>
 </link>
-<joint name="continuous_revolute 2" type="continuous">
+<joint name="continuous_revolute_2" type="continuous">
 <origin xyz="1.1102230246251565404e-16 -0.35000000000000003331 -0.024999999999999994449" rpy="3.141592653589793116 -6.1629758220391519929e-33 3.141592653589793116" />
 <parent link="cart_swinger" />
@@ -148,5 +150,5 @@
 <joint_properties friction="0.0"/>
 </joint>
-<joint name="continuous_revolute 1" type="continuous">
+<joint name="continuous_revolute_1" type="continuous">
 <origin xyz="0 -0.064682458365518544219 5.5511151231257827021e-17" rpy="-1.570796326794896558 -3.0839528461809912666e-16 2.5386489872101804252e-48" />
 <parent link="cart_move" />
